Commit message: changed vehicle to ATV

File: src/sim/smb_simulator/smb_description/urdf/smb.urdf.xacro (robot description, xacro)
@@ -5,8 +5,8 @@
 	<xacro:arg name="robot_namespace" default="/" />
 	<xacro:property name="M_PI" value="3.14159"/>
-	<xacro:property name="chassisHeight" value="0.22"/>
-	<xacro:property name="chassisLength" value="0.605"/>
-	<xacro:property name="chassisWidth" value="0.410"/>
-	<xacro:property name="chassisMass" value="40"/>
+	<xacro:property name="chassisHeight" value="1.26"/>
+	<xacro:property name="chassisLength" value="2.184"/>
+	<xacro:property name="chassisWidth" value="1.168"/>
+	<xacro:property name="chassisMass" value="200.0"/>
 	<!-- Included URDF/XACRO Files -->
 	<xacro:include filename="$(find smb_description)/urdf/wheel.urdf.xacro" />
@@ -14,15 +14,8 @@
 	<!-- Base link is the robot chassis -->
 	<link name="base_link">
-		<!-- <visual>
-			<origin xyz="0 0 0" rpy="0 0 0" />
+		<visual>
+			<origin xyz="0.05 0 0.05"/>
 			<geometry>
-				<box size="${chassisLength} ${chassisWidth} ${chassisHeight}"/>
-			</geometry>
-			<material name="blue"/>
-		</visual> -->
-		<visual>
-			<origin xyz="0.423 0.42 -0.25" rpy="1.57 0 -1.57" />
-			<geometry>
-				<mesh filename="package://smb_description/meshes/SMB_COARSE.dae" scale="0.001 0.001 0.001" />
+				<mesh filename="package://smb_description/meshes/rigid_body.stl" scale="0.001 0.001 0.001" />
 			</geometry>
 			<material name="w">
@@ -33,5 +26,5 @@
 			<origin xyz="0 0 0" rpy="0 0 0" />
 			<geometry>
-				<box size="${chassisLength} ${chassisWidth} ${chassisHeight}"/>
+				<mesh filename="package://smb_description/meshes/rigid_body.stl" scale="0.001 0.001 0.001" />
 			</geometry>
 		</collision>
@@ -55,14 +48,14 @@
 	<!-- SMB wheel macros -->
 	<xacro:smb_wheel wheel_prefix="LF">
-		<origin xyz="${frontWheelX} ${chassisWidth/2+wheelClearance+wheelWidth/2} ${-wheelHeight}" rpy="0 0 0" />
+		<origin xyz="${frontWheelX} ${chassisWidth/2+wheelClearance-wheelWidth/2} ${-wheelHeight}" rpy="0 0 0" />
 	</xacro:smb_wheel>
 	<xacro:smb_wheel wheel_prefix="RF">
-		<origin xyz="${frontWheelX} ${-chassisWidth/2-wheelClearance-wheelWidth/2} ${-wheelHeight}" rpy="0 0 0" />
+		<origin xyz="${frontWheelX} ${-chassisWidth/2-wheelClearance+wheelWidth/2} ${-wheelHeight}" rpy="0 0 0" />
 	</xacro:smb_wheel>
 	<xacro:smb_wheel wheel_prefix="LH">
-		<origin xyz="${backWheelX} ${chassisWidth/2+wheelClearance+wheelWidth/2} ${-wheelHeight}" rpy="0 0 0" />
+		<origin xyz="${backWheelX} ${chassisWidth/2+wheelClearance-wheelWidth/2} ${-wheelHeight}" rpy="0 0 0" />
 	</xacro:smb_wheel>
 	<xacro:smb_wheel wheel_prefix="RH">
-		<origin xyz="${backWheelX} ${-chassisWidth/2-wheelClearance-wheelWidth/2} ${-wheelHeight}" rpy="0 0 0" />
+		<origin xyz="${backWheelX} ${-chassisWidth/2-wheelClearance+wheelWidth/2} ${-wheelHeight}" rpy="0 0 0" />
 	</xacro:smb_wheel>
 	<!-- ROS control plugin to move the robot in simulation -->
@@ -82,7 +75,8 @@
 		</plugin>
 	</gazebo>
-	<xacro:include filename="$(find smb_description)/urdf/sensor_head.urdf.xacro"/>
-	<xacro:sensor_head parent="base_link" name="sensor_head">
-		<origin xyz="0.2 0 0.576" rpy="0 0 0" />
-	</xacro:sensor_head>
+	<xacro:arg name="gpu" default="true"/>
+	<xacro:include filename="$(find lidar_description)/urdf/VLP-16.urdf.xacro"/>
+	<xacro:VLP-16 parent="base_link" name="velodyne" topic="velodyne_points" hz="10" samples="440" gpu="$(arg gpu)" collision_range="1.5" min_range="1.5">
+		<origin xyz="0.835 0.02 0.44" rpy="0 0 0" />
+	</xacro:VLP-16>
 </robot>

File: src/sim/smb_simulator/smb_description/urdf/wheel.urdf.xacro (robot description, xacro)
@@ -3,11 +3,11 @@
     <xacro:property name="PI" value="3.1415926535897931"/>
     <xacro:property name="robot_name" value="smb"/>
-    <xacro:property name="wheelWidth" value="0.185"/>
-    <xacro:property name="wheelRadius" value="0.19"/>
-    <xacro:property name="frontWheelX" value="0.2159"/>
-    <xacro:property name="backWheelX" value="-0.21"/>
-    <xacro:property name="wheelClearance" value="0.03"/>
-    <xacro:property name="wheelHeight" value="0.05"/>
-    <xacro:property name="wheelMass" value="5"/>
+    <xacro:property name="wheelWidth" value="0.356"/>
+    <xacro:property name="wheelRadius" value="0.347311"/>
+    <xacro:property name="frontWheelX" value="0.75"/>
+    <xacro:property name="backWheelX" value="-0.75"/>
+    <xacro:property name="wheelClearance" value="0.02"/>
+    <xacro:property name="wheelHeight" value="0.425"/>
+    <xacro:property name="wheelMass" value="0.5"/>
 	<xacro:macro name="smb_wheel" params="wheel_prefix *joint_pose">
 		<link name="${wheel_prefix}_WHEEL_LINK">
@@ -18,8 +18,9 @@
 			</inertial>
 			<visual>
-				<origin xyz="0 0 0" rpy="${M_PI/2} 0 0" />
+				<origin xyz="0 0 0" rpy="0 0 0" />
 				<geometry>
-					<!-- <cylinder length="${wheelWidth}" radius="${wheelRadius}"/> -->
-					<cylinder length="0.17" radius="0.20"/>  <!-- wheel visual dimensions are small to make the mesh fit properly -->
+					<!-- <mesh filename="package://smb_description/meshes/${wheel_prefix}_wheel.stl" scale="0.001 0.001 0.001"/> -->
+					<cylinder length="${wheelWidth}" radius="${wheelRadius}"/>
+					<!-- <cylinder length="0.17" radius="0.20"/>  wheel visual dimensions are small to make the mesh fit properly -->
 				</geometry>
 				<material name="black"/>
@@ -28,4 +29,5 @@
 				<origin xyz="0 0 0" rpy="${M_PI/2} 0 0" />
 				<geometry>
+					<!-- <mesh filename="package://smb_description/meshes/{wheel_prefix}_wheel.stl" scale="0.001 0.001 0.001"/> -->
 					<cylinder length="${wheelWidth}" radius="${wheelRadius}" />
 				</geometry>

Commit message: Updated launch file to maze_world map and correct spawn location for ATV. Configured wheels and weight of ATV

File: src/sim/smb_simulator/smb_description/urdf/smb.urdf.xacro (robot description, xacro)
@@ -8,5 +8,5 @@
 	<xacro:property name="chassisLength" value="2.184"/>
 	<xacro:property name="chassisWidth" value="1.168"/>
-	<xacro:property name="chassisMass" value="200.0"/>
+	<xacro:property name="chassisMass" value="300.0"/>
 	<!-- Included URDF/XACRO Files -->
 	<xacro:include filename="$(find smb_description)/urdf/wheel.urdf.xacro" />

File: src/sim/smb_simulator/smb_description/urdf/wheel.urdf.xacro (robot description, xacro)
@@ -9,5 +9,5 @@
     <xacro:property name="wheelClearance" value="0.02"/>
     <xacro:property name="wheelHeight" value="0.425"/>
-    <xacro:property name="wheelMass" value="0.5"/>
+    <xacro:property name="wheelMass" value="10.0"/>
 	<xacro:macro name="smb_wheel" params="wheel_prefix *joint_pose">
 		<link name="${wheel_prefix}_WHEEL_LINK">
@@ -18,5 +18,5 @@
 			</inertial>
 			<visual>
-				<origin xyz="0 0 0" rpy="0 0 0" />
+				<origin xyz="0 0 0" rpy="${M_PI/2} 0 0" />
 				<geometry>
 					<!-- <mesh filename="package://smb_description/meshes/${wheel_prefix}_wheel.stl" scale="0.001 0.001 0.001"/> -->
