Commit message: changed values in planner_control_interface_sim_config.yaml in RobotDynamics to higher velocity values

File: src/sim/smb_simulator/smb_description/urdf/wheel.urdf.xacro (robot description, xacro)
@@ -9,5 +9,5 @@
     <xacro:property name="wheelClearance" value="0.02"/>
     <xacro:property name="wheelHeight" value="0.425"/>
-    <xacro:property name="wheelMass" value="0.5"/>
+    <xacro:property name="wheelMass" value="10.0"/>
 	<xacro:macro name="smb_wheel" params="wheel_prefix *joint_pose">
 		<link name="${wheel_prefix}_WHEEL_LINK">
@@ -18,5 +18,5 @@
 			</inertial>
 			<visual>
-				<origin xyz="0 0 0" rpy="0 0 0" />
+				<origin xyz="0 0 0" rpy="${M_PI/2} 0 0" />
 				<geometry>
 					<!-- <mesh filename="package://smb_description/meshes/${wheel_prefix}_wheel.stl" scale="0.001 0.001 0.001"/> -->
@@ -35,6 +35,6 @@
 		</link>
 		<gazebo reference="${wheel_prefix}_WHEEL_LINK">
-			<mu1 value="1.0"/>
-			<mu2 value="1.0"/>
+			<mu1 value="100000000000.0"/>
+			<mu2 value="100000000000.0"/>
 			<kp value="10000000.0" />
 			<kd value="1.0" />
