Commit message: updated parameters and settings

File: src/sim/lonewolf_sim/atv_description/urdf/atv.urdf.xacro (robot description, xacro)
@@ -25,7 +25,11 @@
 		</visual>
 		<collision>
-			<origin xyz="0 0 0" rpy="0 0 0" />
+			<!-- <origin xyz="0 0 0" rpy="0 0 0" />
 			<geometry>
 				<box size="${chassisLength} ${chassisWidth} ${chassisHeight}"/>
+			</geometry> -->
+            <origin xyz="0 0 0" rpy="0 0 0" />
+			<geometry>
+				<mesh filename="package://atv_description/meshes/rigid_body.stl" scale="0.001 0.001 0.001" />
 			</geometry>
 		</collision>

Commit message: changed collison back to mesh

File: src/sim/lonewolf_sim/atv_description/urdf/atv.urdf.xacro (robot description, xacro)
@@ -24,14 +24,18 @@
 			</material>
 		</visual>
-		<collision>
-			<!-- <origin xyz="0 0 0" rpy="0 0 0" />
+        <!-- Box collision -->
+		<!-- <collision>
+			<origin xyz="0 0 0" rpy="0 0 0" />
 			<geometry>
 				<box size="${chassisLength} ${chassisWidth} ${chassisHeight}"/>
-			</geometry> -->
-            <origin xyz="0 0 0" rpy="0 0 0" />
+			</geometry>
+		</collision> -->
+        <!-- Mesh collision -->
+        <collision>
+        <origin xyz="0 0 0" rpy="0 0 0" />
 			<geometry>
 				<mesh filename="package://atv_description/meshes/rigid_body.stl" scale="0.001 0.001 0.001" />
 			</geometry>
-		</collision>
+        </collision>
 	</link>
 	<gazebo reference="base_link">
